File: Main PCB/Sensor.kicad_sch (KiCad schematic)
At the start: 222 parts, among them U10 SLSS49E-3, U11 SLSS49E-3, U12 SLSS49E-3, U13 SLSS49E-3, U14 SLSS49E-3, U15 SLSS49E-3, U16 SLSS49E-3, U17 SLSS49E-3, U18 SLSS49E-3, U19 SLSS49E-3, U20 SLSS49E-3, U21 SLSS49E-3, U22 SLSS49E-3, U23 SLSS49E-3, U24 SLSS49E-3, U25 SLSS49E-3, U26 SLSS49E-3, U27 SLSS49E-3, U28 SLSS49E-3, U29 SLSS49E-3, U30 SLSS49E-3, U31 SLSS49E-3, U32 SLSS49E-3, U33 SLSS49E-3, U34 SLSS49E-3, U35 SLSS49E-3, U36 SLSS49E-3, U37 SLSS49E-3, U38 SLSS49E-3, U39 SLSS49E-3, U40 SLSS49E-3, U41 SLSS49E-3, U42 SLSS49E-3, U43 SLSS49E-3, U44 SLSS49E-3, U45 SLSS49E-3, U46 SLSS49E-3, U47 SLSS49E-3, U48 SLSS49E-3, U49 SLSS49E-3, U50 SLSS49E-3, U51 SLSS49E-3, U52 SLSS49E-3, U53 SLSS49E-3, U54 SLSS49E-3, U55 SLSS49E-3, U56 SLSS49E-3, U57 SLSS49E-3, U58 SLSS49E-3, U59 SLSS49E-3, U6 SLSS49E-3, U60 SLSS49E-3, U61 SLSS49E-3, U62 SLSS49E-3, U63 SLSS49E-3, U64 SLSS49E-3, U65 SLSS49E-3, U66 SLSS49E-3, U67 SLSS49E-3, U68 SLSS49E-3, U69 SLSS49E-3, U7 SLSS49E-3, U70 SLSS49E-3, U71 SLSS49E-3, U72 SLSS49E-3, U73 SLSS49E-3, U74 SLSS49E-3, U75 SLSS49E-3, U76 SLSS49E-3, U77 SLSS49E-3, U78 SLSS49E-3, U79 SLSS49E-3, U8 SLSS49E-3, U80 SLSS49E-3, U81 SLSS49E-3, U82 SLSS49E-3, U83 SLSS49E-3, U84 SLSS49E-3, U85 SLSS49E-3, U86 SLSS49E-3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

Commit message: Small fix
Parts:
- U49: footprint Hall_Sensor_Keyboard:SLSS49E_MX_2.25U-ReversedStabilizers -> Hall_Sensor_Keyboard:SLSS49E_MX_2.25U
Changed lines of the file:
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@@
 			)
 		)
-		(property "Footprint" "Hall_Sensor_Keyboard:SLSS49E_MX_2.25U-ReversedStabilizers"
+		(property "Footprint" "Hall_Sensor_Keyboard:SLSS49E_MX_2.25U"
 			(at 323.85 119.38 0)
 			(effects
